File: Hardware/Digital_LC_Meter.sch (KiCad schematic (older format))
At the start: 25 parts

Commit message: Converted schematic to KicadV5
Parts:
- removed C_BP1: 100nF, Capacitors_THT:C_Rect_L7.0mm_W2.0mm_P5.00mm, symbol C
- removed C_CAL1, C_CAL2: 1nF 1%, Capacitors_THT:C_Disc_D16.0mm_W5.0mm_P7.50mm, symbol C
- removed C_CP1, C_OSC1: 10uF Tant, Capacitors_THT:CP_Radial_Tantal_D5.0mm_P5.00mm, symbol CP
- removed D_IMP1: 1N4148, Diodes_THT:D_DO-35_SOD27_P7.62mm_Horizontal, symbol D
- removed J_CAL_ERASE1, J_CAL_LK1, J_DUT1, J_PWR1, J_RESET1: Conn_01x02, Pin_Headers:Pin_Header_Straight_1x02_Pitch2.54mm, symbol Conn_01x02
- removed J_FUNCSEL1: Conn_01x06, Pin_Headers:Pin_Header_Straight_1x06_Pitch2.54mm, symbol Conn_01x06
- removed J_LCD_OLED1: Conn_01x04, Pin_Headers:Pin_Header_Straight_1x04_Pitch2.54mm, symbol Conn_01x04
- removed J_NANO_TX1, J_NANO_VIN1: Conn_01x15, Pin_Headers:Pin_Header_Straight_1x15_Pitch2.54mm, symbol Conn_01x15
- removed J_NUDGECAL1: Conn_01x03, Pin_Headers:Pin_Header_Straight_1x03_Pitch2.54mm, symbol Conn_01x03
- removed K_CAL1: G5Q-1A, Relays_THT:Relay_SPST_OMRON-G5Q, symbol G5Q-1A
- removed L_CAL1: 100uH, Inductors_THT:L_Radial_D8.7mm_P5.00mm_Fastron_07HCP, symbol L_Core_Ferrite_Small
- removed R_FOUT1: 6K8, Resistors_THT:R_Axial_DIN0207_L6.3mm_D2.5mm_P7.62mm_Horizontal, symbol R
- removed R_NBIAS1, R_PBIAS1, R_PF1: 100K, Resistors_THT:R_Axial_DIN0207_L6.3mm_D2.5mm_P7.62mm_Horizontal, symbol R
- removed R_OSC1: 47K, Resistors_THT:R_Axial_DIN0207_L6.3mm_D2.5mm_P7.62mm_Horizontal, symbol R
- removed R_PBIAS2: 4K7, Resistors_THT:R_Axial_DIN0207_L6.3mm_D2.5mm_P7.62mm_Horizontal, symbol R
- removed U_OSC1: LM311, Housings_DIP:DIP-8_W7.62mm_Socket, symbol LM311
- added C_BP1: 100nF, Capacitor_THT:C_Rect_L7.0mm_W2.0mm_P5.00mm, symbol Device:C
- added C_COUP1, C_OSC1: 10uF, Capacitor_THT:CP_Radial_D5.0mm_P2.50mm, symbol Device:CP
- added C_MICA1, C_MICA2: 1nF, Capacitor_THT:C_Rect_L7.0mm_W2.0mm_P5.00mm, symbol Device:C
- added D1: 1N4148, Diode_THT:D_DO-35_SOD27_P7.62mm_Horizontal, symbol Device:D
- added J_CALJUMPER1, J_ERASEBTN1, J_INPUT1, J_PWR1, J_RESETBTN1: Conn_01x02, Connector_PinHeader_2.54mm:PinHeader_1x02_P2.54mm_Vertical, symbol Connector_Generic:Conn_01x02
- added J_LCSELECTSPDT1: Conn_01x06, Connector_PinHeader_2.54mm:PinHeader_1x06_P2.54mm_Vertical, symbol Connector_Generic:Conn_01x06
- added J_NANOTX1, J_NANOVIN1: Conn_01x15, Connector_PinHeader_2.54mm:PinHeader_1x15_P2.54mm_Vertical, symbol Connector_Generic:Conn_01x15
- added J_NUDGEBTN1: Conn_01x03, Connector_PinHeader_2.54mm:PinHeader_1x03_P2.54mm_Vertical, symbol Connector_Generic:Conn_01x03
- added J_OLED1: Conn_01x04, Connector_PinHeader_2.54mm:PinHeader_1x04_P2.54mm_Vertical, symbol Connector_Generic:Conn_01x04
- added K1: G5Q-1A, Relay_THT:Relay_SPST_Omron-G5Q-1A, symbol Relay:G5Q-1A
- added L1: 100uH, Inductor_THT:L_Radial_D7.8mm_P5.00mm_Fastron_07HCP, symbol Device:L_Core_Ferrite_Small
- added R3, R_BIAS1, R_BIAS2: 100K, Resistor_THT:R_Axial_DIN0207_L6.3mm_D2.5mm_P7.62mm_Horizontal, symbol Device:R
- added R_BIAS3: 4K7, Resistor_THT:R_Axial_DIN0207_L6.3mm_D2.5mm_P7.62mm_Horizontal, symbol Device:R
- added R_OSC1: 47K, Resistor_THT:R_Axial_DIN0207_L6.3mm_D2.5mm_P7.62mm_Horizontal, symbol Device:R
- added R_SIG1: 6K8, Resistor_THT:R_Axial_DIN0207_L6.3mm_D2.5mm_P7.62mm_Horizontal, symbol Device:R
- added U_OSC1: LM311, Package_DIP:DIP-8_W7.62mm_Socket, symbol Comparator:LM311
Connections:
- wire segments 79 -> 93

Commit message: updated kicad files
Parts:
- removed D1: 1N4148, Diode_THT:D_DO-35_SOD27_P7.62mm_Horizontal, symbol Device:D
- removed K1: G5Q-1A, Relay_THT:Relay_SPST_Omron-G5Q-1A, symbol Relay:G5Q-1A
- added J_DA1, J_DK1: Conn_01x01, Connector_PinHeader_2.54mm:PinHeader_1x01_P2.54mm_Vertical, symbol Connector_Generic:Conn_01x01
- added U_RLY1: TE_ReedRelay_V23100V4xxxA010, TE_Reed_Relay_V23100V4:TE_ReedRelay_V23100V4, symbol TE_ReedRelay_V23100V4:TE_ReedRelay_V23100V4xxxA010
Connections:
- wire segments 93 -> 97
- no-connect marks 17 -> 20
Changed lines of the file:
@@
 Wire Wire Line
 	3025 2750 4025 2750
-Wire Wire Line
-	8450 5825 8450 6125
-Text Label 8450 6125 1    60   ~ 0
-GND
-Wire Wire Line
-	8850 5825 8850 6125
 Text Label 8850 6125 1    60   ~ 0
 GND
@@
 DPDT:\nUP1\nDOWN1\nIN1\nIN2\nUP2\nDOWN2
 Wire Wire Line
-	9550 5700 9550 6125
+	9550 5875 9550 6125
 Text Label 9550 6125 1    60   ~ 0
 GND
 Wire Wire Line
-	9550 5400 9550 5000
-Wire Wire Line
-	8850 5000 9550 5000
-Wire Wire Line
-	8850 5000 8850 5225
-Connection ~ 9550 5000
-Text Label 10400 5000 2    60   ~ 0
+	9550 5150 9550 4800
+Wire Wire Line
+	8850 4800 9550 4800
+Connection ~ 9550 4800
+Text Label 10400 4800 2    60   ~ 0
 RELAY_PIN3
 Wire Wire Line
@@
 GND
 Wire Wire Line
-	8450 5225 8450 4800
-Wire Wire Line
-	8450 4800 4475 4800
+	8650 4800 4475 4800
 Wire Wire Line
 	4475 4800 4475 3775
@@
 	4025 2750 4475 2750
 Wire Wire Line
-	9550 5000 10400 5000
+	9550 4800 10400 4800
 Wire Wire Line
 	7125 3700 7125 3875
@@
 $EndComp
 $Comp
-L Device:D D1
-U 1 1 5B978454
-P 9550 5550
-F 0 "D1" V 9504 5629 50  0000 L CNN
-F 1 "1N4148" V 9595 5629 50  0000 L CNN
-F 2 "Diode_THT:D_DO-35_SOD27_P7.62mm_Horizontal" H 9550 5550 50  0001 C CNN
-F 3 "~" H 9550 5550 50  0001 C CNN
-	1    9550 5550
-	0    1    1    0
-$EndComp
-$Comp
 L Comparator:LM311 U_OSC1
 U 1 1 5B978CA1
@@
 	1    6375 2850
 	1    0    0    -1
-$EndComp
-$Comp
-L Relay:G5Q-1A K1
-U 1 1 5B979EA0
-P 8650 5525
-F 0 "K1" H 8220 5571 50  0000 R CNN
-F 1 "G5Q-1A" H 8220 5480 50  0000 R CNN
-F 2 "Relay_THT:Relay_SPST_Omron-G5Q-1A" H 9000 5475 50  0001 L CNN
-F 3 "https://www.omron.com/ecb/products/pdf/en-g5q.pdf" H 9750 5225 50  0001 C CNN
-	1    8650 5525
-	-1   0    0    -1
 $EndComp
 $Comp
@@
 	0    -1   -1   0
 $EndComp
+$Comp
+L TE_ReedRelay_V23100V4:TE_ReedRelay_V23100V4xxxA010 U_RLY1
+U 1 1 5B996138
+P 8800 5475
+F 0 "U_RLY1" H 8450 5400 60  0000 R CNN
+F 1 "TE_ReedRelay_V23100V4xxxA010" H 8450 5575 60  0000 R CNN
+F 2 "TE_Reed_Relay_V23100V4:TE_ReedRelay_V23100V4" H 8800 5455 60  0001 C CNN
+F 3 "" H 8800 5455 60  0001 C CNN
+	1    8800 5475
+	1    0    0    1
+$EndComp
+$Comp
+L Connector_Generic:Conn_01x01 J_DK1
+U 1 1 5B9A08C2
+P 9550 5350
+F 0 "J_DK1" V 9425 5430 50  0000 L CNN
+F 1 "Conn_01x01" V 9514 5430 50  0000 L CNN
+F 2 "Connector_PinHeader_2.54mm:PinHeader_1x01_P2.54mm_Vertical" H 9550 5350 50  0001 C CNN
+F 3 "~" H 9550 5350 50  0001 C CNN
+	1    9550 5350
+	0    1    1    0
+$EndComp
+$Comp
+L Connector_Generic:Conn_01x01 J_DA1
+U 1 1 5B9A3151
+P 9550 5675
+F 0 "J_DA1" V 9515 5588 50  0000 R CNN
+F 1 "Conn_01x01" V 9426 5588 50  0000 R CNN
+F 2 "Connector_PinHeader_2.54mm:PinHeader_1x01_P2.54mm_Vertical" H 9550 5675 50  0001 C CNN
+F 3 "~" H 9550 5675 50  0001 C CNN
+	1    9550 5675
+	0    -1   -1   0
+$EndComp
+Wire Wire Line
+	8750 5850 8850 5850
+Connection ~ 8850 5850
+Wire Wire Line
+	8850 5850 8850 6125
+Wire Wire Line
+	8950 5850 8850 5850
+NoConn ~ 8950 5175
+NoConn ~ 8750 5175
+NoConn ~ 8650 5775
+Wire Wire Line
+	8850 4800 8850 5175
+Wire Wire Line
+	8650 5175 8650 4800
+Wire Wire Line
+	8750 5775 8750 5850
+Wire Wire Line
+	8850 5775 8850 5850
+Wire Wire Line
+	8950 5775 8950 5850
 $EndSCHEMATC

Commit message: Added 2nd OLED and TCA9548A IICMux. Updated Schematic and Board Layouts
Parts:
- added J_IICMUX_SC7, J_IICMUX_VIN1: Conn_01x12, Connector_PinHeader_2.54mm:PinHeader_1x12_P2.54mm_Vertical, symbol Connector_Generic:Conn_01x12
- added J_OLED2: Conn_01x04, Connector_PinHeader_2.54mm:PinHeader_1x04_P2.54mm_Vertical, symbol Connector_Generic:Conn_01x04
Connections:
- net labels added: SCL0, SCL1, SDA0, SDA1
- wire segments 97 -> 117
- no-connect marks 20 -> 32
Other:
- note added: "SC7\nSD7\nSC6\nSD6\nSC5\nSD5\nSC4\nSD4\nSC3\nSD3\nSC2\nSD2"
- note added: "TCA9548A\nPin Mappings:"
- note added: "VIN\nGND\nSDA\nSCL\nRST\nA0\nA1\nA2\nSD0\nSC0\nSD1\nSC1"
Changed lines of the file:
@@
 Comment4 ""
 $EndDescr
-Text Notes 8775 3200 0    63   ~ 0
+Text Notes 8875 2525 0    63   ~ 0
 TX\nRX\nRST\nGND\n2\n3\n4\n5\n6\n7\n8\n9\n10\n11\n12
-Text Notes 9750 3200 0    63   ~ 0
+Text Notes 9800 2525 0    63   ~ 0
 VIN\nGND\nRST\n5V\n21\n20\n19\n18\n17\n16\n15\n14\nAREF\n3V3\n13\n
 Wire Wire Line
@@
 GND
 Wire Wire Line
-	10250 1775 10475 1775
-Text Label 10475 1775 0    60   ~ 0
+	10300 1100 10525 1100
+Text Label 10525 1100 0    60   ~ 0
 VIN
 Wire Wire Line
-	10250 1875 10475 1875
-Text Label 10475 1875 0    60   ~ 0
+	10300 1200 10525 1200
+Text Label 10525 1200 0    60   ~ 0
 GND
 Wire Wire Line
 	1625 6150 1375 6150
 Text Label 1375 6150 0    60   ~ 0
-SDA
+SDA0
 Wire Wire Line
 	1625 6250 1375 6250
 Text Label 1375 6250 0    60   ~ 0
-SCL
+SCL0
 Wire Wire Line
 	1625 6350 1375 6350
@@
 5V
 Wire Wire Line
-	10250 2075 10475 2075
-Text Label 10475 2075 0    60   ~ 0
+	10300 1400 10525 1400
+Text Label 10525 1400 0    60   ~ 0
 5V
 Wire Wire Line
-	10250 2475 10475 2475
-Text Label 10475 2475 0    60   ~ 0
+	10300 1800 10525 1800
+Text Label 10525 1800 0    60   ~ 0
 SDA
 Wire Wire Line
-	10250 2375 10475 2375
-Text Label 10475 2375 0    60   ~ 0
+	10300 1700 10525 1700
+Text Label 10525 1700 0    60   ~ 0
 SCL
 Wire Wire Line
@@
 CL_BAR_PIN2
 Wire Wire Line
-	8500 2175 7725 2175
-Text Label 7725 2175 0    60   ~ 0
+	8600 1500 7825 1500
+Text Label 7825 1500 0    60   ~ 0
 CL_BAR_PIN2
 Text Notes 2550 4475 0    63   ~ 0
@@
 RELAY_PIN3
 Wire Wire Line
-	8500 2275 7725 2275
-Text Label 7725 2275 0    60   ~ 0
+	8600 1600 7825 1600
+Text Label 7825 1600 0    60   ~ 0
 RELAY_PIN3
 Wire Wire Line
-	8500 2575 7725 2575
-Text Label 7725 2575 0    60   ~ 0
+	8600 1900 7825 1900
+Text Label 7825 1900 0    60   ~ 0
 INCR_PIN6
-Text Label 7725 2375 0    60   ~ 0
+Text Label 7825 1700 0    60   ~ 0
 DECR_PIN4
 Wire Wire Line
-	8500 2375 7725 2375
+	8600 1700 7825 1700
 Connection ~ 7125 3700
 Wire Wire Line
@@
 OSC_SIG_PIN5
 Wire Wire Line
-	8500 2475 7725 2475
-Text Label 7725 2475 0    60   ~ 0
+	8600 1800 7825 1800
+Text Label 7825 1800 0    60   ~ 0
 OSC_SIG_PIN5
 Wire Wire Line
-	8500 2675 7725 2675
-Text Label 7725 2675 0    60   ~ 0
+	8600 2000 7825 2000
+Text Label 7825 2000 0    60   ~ 0
 CAL_LK_PIN7
 Wire Wire Line
-	8500 2775 7725 2775
-Text Label 7725 2775 0    60   ~ 0
+	8600 2100 7825 2100
+Text Label 7825 2100 0    60   ~ 0
 CAL_ERASE_PIN8
 Wire Wire Line
@@
 Connection ~ 2300 1450
 Wire Wire Line
-	10250 1975 10475 1975
-Text Label 10475 1975 0    60   ~ 0
+	10300 1300 10525 1300
+Text Label 10525 1300 0    60   ~ 0
 RESET_PIN
 Wire Wire Line
@@
 Text Label 4825 7250 0    60   ~ 0
 GND
-NoConn ~ 8500 1775
-NoConn ~ 8500 1875
-NoConn ~ 8500 1975
-NoConn ~ 8500 2075
-NoConn ~ 8500 2875
-NoConn ~ 8500 2975
-NoConn ~ 8500 3075
-NoConn ~ 8500 3175
-NoConn ~ 10250 3175
-NoConn ~ 10250 3075
-NoConn ~ 10250 2975
-NoConn ~ 10250 2875
-NoConn ~ 10250 2775
-NoConn ~ 10250 2675
-NoConn ~ 10250 2575
-NoConn ~ 10250 2175
-NoConn ~ 10250 2275
-Text Notes 9000 1675 0    60   ~ 0
+NoConn ~ 8600 1100
+NoConn ~ 8600 1200
+NoConn ~ 8600 1300
+NoConn ~ 8600 1400
+NoConn ~ 8600 2200
+NoConn ~ 8600 2300
+NoConn ~ 8600 2400
+NoConn ~ 8600 2500
+NoConn ~ 10300 2500
+NoConn ~ 10300 2400
+NoConn ~ 10300 2300
+NoConn ~ 10300 2200
+NoConn ~ 10300 2100
+NoConn ~ 10300 2000
+NoConn ~ 10300 1900
+NoConn ~ 10300 1500
+NoConn ~ 10300 1600
+Text Notes 9050 1000 0    60   ~ 0
 Arduino Nano\nPin Mappings:
 Wire Wire Line
@@
 L Connector_Generic:Conn_01x15 J_NANOTX1
 U 1 1 5B972B1E
-P 8700 2475
-F 0 "J_NANOTX1" H 8700 1625 50  0000 L CNN
-F 1 "Conn_01x15" H 8675 1550 50  0000 L CNN
-F 2 "Connector_PinHeader_2.54mm:PinHeader_1x15_P2.54mm_Vertical" H 8700 2475 50  0001 C CNN
-F 3 "~" H 8700 2475 50  0001 C CNN
-	1    8700 2475
+P 8800 1800
+F 0 "J_NANOTX1" H 8550 2775 50  0000 L CNN
+F 1 "Conn_01x15" H 8550 2675 50  0000 L CNN
+F 2 "Connector_PinHeader_2.54mm:PinHeader_1x15_P2.54mm_Vertical" H 8800 1800 50  0001 C CNN
+F 3 "~" H 8800 1800 50  0001 C CNN
+	1    8800 1800
 	1    0    0    -1
 $EndComp
@@
 L Connector_Generic:Conn_01x15 J_NANOVIN1
 U 1 1 5B972BA3
-P 10050 2475
-F 0 "J_NANOVIN1" H 10050 1625 50  0000 C CNN
-F 1 "Conn_01x15" H 10050 1550 50  0000 C CNN
-F 2 "Connector_PinHeader_2.54mm:PinHeader_1x15_P2.54mm_Vertical" H 10050 2475 50  0001 C CNN
-F 3 "~" H 10050 2475 50  0001 C CNN
-	1    10050 2475
+P 10100 1800
+F 0 "J_NANOVIN1" H 10100 2775 50  0000 C CNN
+F 1 "Conn_01x15" H 10100 2675 50  0000 C CNN
+F 2 "Connector_PinHeader_2.54mm:PinHeader_1x15_P2.54mm_Vertical" H 10100 1800 50  0001 C CNN
+F 3 "~" H 10100 1800 50  0001 C CNN
+	1    10100 1800
 	-1   0    0    -1
 $EndComp
@@
 Wire Wire Line
 	8950 5775 8950 5850
+$Comp
+L Connector_Generic:Conn_01x12 J_IICMUX_SC7
+U 1 1 5B999C08
+P 10100 3500
+F 0 "J_IICMUX_SC7" H 10020 4217 50  0000 C CNN
+F 1 "Conn_01x12" H 10020 4126 50  0000 C CNN
+F 2 "Connector_PinHeader_2.54mm:PinHeader_1x12_P2.54mm_Vertical" H 10100 3500 50  0001 C CNN
+F 3 "~" H 10100 3500 50  0001 C CNN
+	1    10100 3500
+	-1   0    0    -1
+$EndComp
+$Comp
+L Connector_Generic:Conn_01x12 J_IICMUX_VIN1
+U 1 1 5B9A71AD
+P 8800 3500
+F 0 "J_IICMUX_VIN1" H 8475 4225 50  0000 L CNN
+F 1 "Conn_01x12" H 8525 4125 50  0000 L CNN
+F 2 "Connector_PinHeader_2.54mm:PinHeader_1x12_P2.54mm_Vertical" H 8800 3500 50  0001 C CNN
+F 3 "~" H 8800 3500 50  0001 C CNN
+	1    8800 3500
+	1    0    0    -1
+$EndComp
+Text Notes 8900 4125 0    63   ~ 0
+VIN\nGND\nSDA\nSCL\nRST\nA0\nA1\nA2\nSD0\nSC0\nSD1\nSC1
+Text Notes 9800 4125 0    63   ~ 0
+SC7\nSD7\nSC6\nSD6\nSC5\nSD5\nSC4\nSD4\nSC3\nSD3\nSC2\nSD2
+Text Notes 9125 2925 0    63   ~ 0
+TCA9548A\nPin Mappings:
+Wire Wire Line
+	8600 3000 8250 3000
+Text Label 8250 3000 0    63   ~ 0
+5V
+Wire Wire Line
+	8600 3200 8250 3200
+Text Label 8250 3200 0    63   ~ 0
+SDA
+Wire Wire Line
+	8600 3300 8250 3300
+Text Label 8250 3300 0    63   ~ 0
+SCL
+Wire Wire Line
+	8600 3400 8250 3400
+Text Label 8250 3400 0    63   ~ 0
+5V
+Text Label 7850 4000 1    63   ~ 0
+GND
+Wire Wire Line
+	7850 3500 7850 3600
+Wire Wire Line
+	7850 3500 8600 3500
+Wire Wire Line
+	8600 3100 7850 3100
+Wire Wire Line
+	7850 3100 7850 3500
+Connection ~ 7850 3500
+Wire Wire Line
+	8600 3600 7850 3600
+Connection ~ 7850 3600
+Wire Wire Line
+	7850 3600 7850 3700
+Wire Wire Line
+	8600 3700 7850 3700
+Connection ~ 7850 3700
+Wire Wire Line
+	7850 3700 7850 4000
+Wire Wire Line
+	1625 6750 1375 6750
+Text Label 1375 6750 0    60   ~ 0
+SDA1
+Wire Wire Line
+	1625 6850 1375 6850
+Text Label 1375 6850 0    60   ~ 0
+SCL1
+Wire Wire Line
+	1625 6950 1375 6950
+Text Label 1375 6950 0    60   ~ 0
+GND
+Wire Wire Line
+	1625 7050 1375 7050
+Text Label 1375 7050 0    60   ~ 0
+5V
+$Comp
+L Connector_Generic:Conn_01x04 J_OLED2
+U 1 1 5B9E0177
+P 1825 6850
+F 0 "J_OLED2" H 1905 6842 50  0000 L CNN
+F 1 "Conn_01x04" H 1905 6751 50  0000 L CNN
+F 2 "Connector_PinHeader_2.54mm:PinHeader_1x04_P2.54mm_Vertical" H 1825 6850 50  0001 C CNN
+F 3 "~" H 1825 6850 50  0001 C CNN
+	1    1825 6850
+	1    0    0    -1
+$EndComp
+Wire Wire Line
+	8600 3800 8100 3800
+Wire Wire Line
+	8600 3900 8100 3900
+Wire Wire Line
+	8600 4000 8100 4000
+Wire Wire Line
+	8600 4100 8100 4100
+Text Label 8100 3800 0    63   ~ 0
+SDA0
+Text Label 8100 3900 0    63   ~ 0
+SCL0
+Text Label 8100 4000 0    63   ~ 0
+SDA1
+Text Label 8100 4100 0    63   ~ 0
+SCL1
+NoConn ~ 10300 3000
+NoConn ~ 10300 3100
+NoConn ~ 10300 3200
+NoConn ~ 10300 3300
+NoConn ~ 10300 3400
+NoConn ~ 10300 3500
+NoConn ~ 10300 3600
+NoConn ~ 10300 3700
+NoConn ~ 10300 3800
+NoConn ~ 10300 3900
+NoConn ~ 10300 4000
+NoConn ~ 10300 4100
 $EndSCHEMATC

Commit message: updates
- Added I2C Mux (TCA9548A) to design
- Initial prototype tested (firmware needs work)
- Created Front Panel Template for enclosure (Hammond 1455T1601)
Parts:
- R_OSC1: footprint Resistor_THT:R_Axial_DIN0207_L6.3mm_D2.5mm_P7.62mm_Horizontal -> Resistor_THT:R_Axial_DIN0207_L6.3mm_D2.5mm_P10.16mm_Horizontal
Connections:
- wire segments 117 -> 119
Changed lines of the file:
@@
 	1325 4125 2275 4125
 Wire Wire Line
-	1325 4225 2275 4225
+	1325 4225 1375 4225
 Text Label 3025 2750 0    60   ~ 0
 IND_PARALLEL
@@
 F 0 "R_OSC1" V 6418 3700 50  0000 C CNN
 F 1 "47K" V 6509 3700 50  0000 C CNN
-F 2 "Resistor_THT:R_Axial_DIN0207_L6.3mm_D2.5mm_P7.62mm_Horizontal" V 6555 3700 50  0001 C CNN
+F 2 "Resistor_THT:R_Axial_DIN0207_L6.3mm_D2.5mm_P10.16mm_Horizontal" V 6555 3700 50  0001 C CNN
 F 3 "~" H 6625 3700 50  0001 C CNN
 	1    6625 3700
@@
 NoConn ~ 10300 4000
 NoConn ~ 10300 4100
+Wire Wire Line
+	1375 4225 1375 4575
+Connection ~ 1375 4225
+Wire Wire Line
+	1375 4225 2275 4225
+Text Label 1375 4575 1    60   ~ 0
+GND
 $EndSCHEMATC

Commit message: fixed OLED screen wiring on prototype, updated schematic and layout
Parts:
- removed J_IICMUX_SC7, J_IICMUX_VIN1: Conn_01x12, Connector_PinHeader_2.54mm:PinHeader_1x12_P2.54mm_Vertical, symbol Connector_Generic:Conn_01x12
- removed J_OLED1, J_OLED2: Conn_01x04, Connector_PinHeader_2.54mm:PinHeader_1x04_P2.54mm_Vertical, symbol Connector_Generic:Conn_01x04
- added J_SSD1309_OLED1: Conn_01x05, Connector_PinHeader_2.54mm:PinHeader_1x05_P2.54mm_Vertical, symbol Connector_Generic:Conn_01x05
Connections:
- net labels added: INCR_PIN10, SRST
- net labels removed: INCR_PIN6, SCL0, SCL1, SDA0, SDA1
- wire segments 119 -> 101
- no-connect marks 32 -> 19
Other:
- note added: "2.42" SSD1309\nwww.diymore.cc"
- note removed: "SC7\nSD7\nSC6\nSD6\nSC5\nSD5\nSC4\nSD4\nSC3\nSD3\nSC2\nSD2"
- note removed: "TCA9548A\nPin Mappings:"
- note removed: "VIN\nGND\nSDA\nSCL\nRST\nA0\nA1\nA2\nSD0\nSC0\nSD1\nSC1"
